File: EtherDue_Mega16U2.sch (KiCad schematic (older format))
At the start: 26 parts, among them IC601 ATMEGA16U2, P601 USB_5PIN_SHELL, X601 12MHz KX-7 20pF

Commit message: Final ERC cleanup, export net file
Parts:
- C303: renamed from 22pF601; value C -> 22pF
- C304: renamed from 22pF602; value C -> 22pF
- renumbered C601 to C301, C602 to C302, C603 to C305, CD1206-S601 to CD1206-S301, D601 to D301, D602 to D302, F601 to F301, IC601 to IC301, ICSP601 to ICSP301, JP601 to JP301, P601 to P301, R601 to R301, R602 to R302, R603 to R303, R604 to R304, R605 to R305, R606 to R306, R607 to R307, R608 to R308, R609 to R309, R610 to R310, X601 to X301, Z601 to Z301, Z602 to Z302
Changed lines of the file:
@@
-EESchema Schematic File Version 2  date Thu 11 Apr 2013 15:52:58 EST
+EESchema Schematic File Version 2  date Thu 11 Apr 2013 16:32:55 EST
 LIBS:power
 LIBS:device
@@
 $Descr A4 11693 8268
 encoding utf-8
-Sheet 6 6
+Sheet 3 6
 Title ""
 Date "11 apr 2013"
@@
 $EndComp
 $Comp
-L R R605
+L R R305
 U 1 1 5164F3AD
 P 9650 5550
-F 0 "R605" V 9730 5550 50  0000 C CNN
+F 0 "R305" V 9730 5550 50  0000 C CNN
 F 1 "2K7" V 9650 5550 50  0000 C CNN
 F 2 "" H 9650 5550 60  0001 C CNN
@@
 $EndComp
 $Comp
-L R R604
+L R R304
 U 1 1 5164F3A2
 P 9250 5300
-F 0 "R604" V 9330 5300 50  0000 C CNN
+F 0 "R304" V 9330 5300 50  0000 C CNN
 F 1 "1K5" V 9250 5300 50  0000 C CNN
 F 2 "" H 9250 5300 60  0001 C CNN
@@
 $EndComp
 $Comp
-L R R608
+L R R308
 U 1 1 515BD664
 P 10000 4200
-F 0 "R608" V 10080 4200 50  0000 C CNN
+F 0 "R308" V 10080 4200 50  0000 C CNN
 F 1 "1K" V 10000 4200 50  0000 C CNN
 F 2 "" H 10000 4200 60  0001 C CNN
@@
 $EndComp
 $Comp
-L R R609
+L R R309
 U 1 1 515BD654
 P 10000 4500
-F 0 "R609" V 10080 4500 50  0000 C CNN
+F 0 "R309" V 10080 4500 50  0000 C CNN
 F 1 "1K" V 10000 4500 50  0000 C CNN
 F 2 "" H 10000 4500 60  0001 C CNN
@@
 $EndComp
 $Comp
-L LED D602
+L LED D302
 U 1 1 515BD64B
 P 9300 4500
-F 0 "D602" H 9300 4600 50  0000 C CNN
+F 0 "D302" H 9300 4600 50  0000 C CNN
 F 1 "YELLOW" H 9300 4400 50  0000 C CNN
 F 2 "" H 9300 4500 60  0001 C CNN
@@
 $EndComp
 $Comp
-L LED D601
+L LED D301
 U 1 1 515BD62A
 P 9300 4200
-F 0 "D601" H 9300 4300 50  0000 C CNN
+F 0 "D301" H 9300 4300 50  0000 C CNN
 F 1 "YELLOW" H 9300 4100 50  0000 C CNN
 F 2 "" H 9300 4200 60  0001 C CNN
@@
 $EndComp
 $Comp
-L R R610
+L R R310
 U 1 1 515BD5FC
 P 11000 4450
-F 0 "R610" V 11080 4450 50  0000 C CNN
+F 0 "R310" V 11080 4450 50  0000 C CNN
 F 1 "10K" V 11000 4450 50  0000 C CNN
 F 2 "" H 11000 4450 60  0001 C CNN
@@
 NoConn ~ 8100 3650
 $Comp
-L R R607
+L R R307
 U 1 1 515BD5C8
 P 10000 3550
-F 0 "R607" V 10080 3550 50  0000 C CNN
+F 0 "R307" V 10080 3550 50  0000 C CNN
 F 1 "1K" V 10000 3550 50  0000 C CNN
 F 2 "" H 10000 3550 60  0001 C CNN
@@
 RESET_CMD
 $Comp
-L R R606
+L R R306
 U 1 1 515BD538
 P 10000 2500
-F 0 "R606" V 10080 2500 50  0000 C CNN
+F 0 "R306" V 10080 2500 50  0000 C CNN
 F 1 "10K" V 10000 2500 50  0000 C CNN
 F 2 "" H 10000 2500 60  0001 C CNN
@@
 RD-
 $Comp
-L R R602
+L R R302
 U 1 1 515BD4B0
 P 2850 4450
-F 0 "R602" V 2930 4450 50  0000 C CNN
+F 0 "R302" V 2930 4450 50  0000 C CNN
 F 1 "22R" V 2850 4450 50  0000 C CNN
 F 2 "" H 2850 4450 60  0001 C CNN
@@
 $EndComp
 $Comp
-L R R601
+L R R301
 U 1 1 515BD4A7
 P 2850 4250
-F 0 "R601" V 2930 4250 50  0000 C CNN
+F 0 "R301" V 2930 4250 50  0000 C CNN
 F 1 "22R" V 2850 4250 50  0000 C CNN
 F 2 "" H 2850 4250 60  0001 C CNN
@@
 NoConn ~ 1200 4450
 $Comp
-L VR Z602
+L VR Z302
 U 1 1 515BD423
 P 1850 4800
-F 0 "Z602" V 1930 4800 50  0000 C CNN
+F 0 "Z302" V 1930 4800 50  0000 C CNN
 F 1 "PGB1010603" V 1750 4800 50  0000 C CNN
 F 2 "" H 1850 4800 60  0001 C CNN
@@
 $EndComp
 $Comp
-L VR Z601
+L VR Z301
 U 1 1 515BD3FE
 P 1550 4800
-F 0 "Z601" V 1630 4800 50  0000 C CNN
+F 0 "Z301" V 1630 4800 50  0000 C CNN
 F 1 "PGB1010603" V 1450 4800 50  0000 C CNN
 F 2 "" H 1550 4800 60  0001 C CNN
@@
 $EndComp
 $Comp
-L C C601
+L C C301
 U 1 1 515BD2FA
 P 2450 3750
-F 0 "C601" H 2500 3850 50  0000 L CNN
+F 0 "C301" H 2500 3850 50  0000 L CNN
 F 1 "100nF" H 2500 3650 50  0000 L CNN
 F 2 "" H 2450 3750 60  0001 C CNN
@@
 $EndComp
 $Comp
-L FUSE F601
+L FUSE F301
 U 1 1 515BD2D5
 P 2000 3500
-F 0 "F601" H 2100 3550 40  0000 C CNN
+F 0 "F301" H 2100 3550 40  0000 C CNN
 F 1 "PTC MF-MSMF050-2 500mA" H 2000 3350 40  0000 C CNN
 F 2 "" H 2000 3500 60  0001 C CNN
@@
 $EndComp
 $Comp
-L USB_5PIN_SHELL P601
+L USB_5PIN_SHELL P301
 U 1 1 515BD282
 P 1000 4300
-F 0 "P601" H 925 4550 60  0000 C CNN
+F 0 "P301" H 925 4550 60  0000 C CNN
 F 1 "USB_5PIN_SHELL" H 1200 3950 60  0001 C CNN
 F 2 "" H 1000 4300 60  0001 C CNN
@@
 $EndComp
 $Comp
-L C C603
+L C C305
 U 1 1 515BD169
 P 4500 4500
-F 0 "C603" H 4550 4600 50  0000 L CNN
+F 0 "C305" H 4550 4600 50  0000 L CNN
 F 1 "1uF" H 4550 4400 50  0000 L CNN
 F 2 "" H 4500 4500 60  0001 C CNN
@@
 $EndComp
 $Comp
-L C C602
+L C C302
 U 1 1 515BD15F
 P 4100 4500
-F 0 "C602" H 4150 4600 50  0000 L CNN
+F 0 "C302" H 4150 4600 50  0000 L CNN
 F 1 "100nF" H 4150 4400 50  0000 L CNN
 F 2 "" H 4100 4500 60  0001 C CNN
@@
 $EndComp
 $Comp
-L C 22pF602
+L C C304
 U 1 1 515BCF9F
 P 4350 3150
-F 0 "22pF602" H 4400 3250 50  0000 L CNN
-F 1 "C" H 4400 3050 50  0000 L CNN
+F 0 "C304" H 4400 3250 50  0000 L CNN
+F 1 "22pF" H 4400 3050 50  0000 L CNN
 F 2 "" H 4350 3150 60  0001 C CNN
 F 3 "" H 4350 3150 60  0001 C CNN
@@
 $EndComp
 $Comp
-L C 22pF601
+L C C303
 U 1 1 515BCF8C
 P 4350 2750
-F 0 "22pF601" H 4400 2850 50  0000 L CNN
-F 1 "C" H 4400 2650 50  0000 L CNN
+F 0 "C303" H 4400 2850 50  0000 L CNN
+F 1 "22pF" H 4400 2650 50  0000 L CNN
 F 2 "" H 4350 2750 60  0001 C CNN
 F 3 "" H 4350 2750 60  0001 C CNN
@@
 $EndComp
 $Comp
-L CRYSTAL X601
+L CRYSTAL X301
 U 1 1 515BCF7E
 P 4900 2950
-F 0 "X601" H 4900 3100 60  0000 C CNN
+F 0 "X301" H 4900 3100 60  0000 C CNN
 F 1 "12MHz KX-7 20pF" H 4900 2800 60  0000 C CNN
 F 2 "" H 4900 2950 60  0001 C CNN
@@
 8PB7
 $Comp
-L M02X02 JP601
+L M02X02 JP301
 U 1 1 515BCEC1
 P 8650 1400
-F 0 "JP601" H 8550 1500 50  0000 C CNN
+F 0 "JP301" H 8550 1500 50  0000 C CNN
 F 1 "M02X02" H 8600 1200 40  0000 C CNN
 F 2 "" H 8650 1400 60  0001 C CNN
@@
 MISO
 $Comp
-L DIODE CD1206-S601
+L DIODE CD1206-S301
 U 1 1 515BCE47
 P 5300 2000
-F 0 "CD1206-S601" H 5300 1850 40  0000 C CNN
+F 0 "CD1206-S301" H 5300 1850 40  0000 C CNN
 F 1 "DIODE" H 5300 1900 40  0000 C CNN
 F 2 "" H 5300 2000 60  0001 C CNN
@@
 $EndComp
 $Comp
-L R R603
+L R R303
 U 1 1 515BCDE2
 P 5100 2000
-F 0 "R603" V 5180 2000 50  0000 C CNN
+F 0 "R303" V 5180 2000 50  0000 C CNN
 F 1 "10K" V 5100 2000 50  0000 C CNN
 F 2 "" H 5100 2000 60  0001 C CNN
@@
 MISO
 $Comp
-L M02X03 ICSP601
+L M02X03 ICSP301
 U 1 1 515BCD62
 P 4300 1650
-F 0 "ICSP601" H 4200 1750 50  0000 C CNN
+F 0 "ICSP301" H 4200 1750 50  0000 C CNN
 F 1 "M02X03" H 4250 1350 40  0000 C CNN
 F 2 "" H 4300 1650 60  0001 C CNN
@@
 $EndComp
 $Comp
-L ATMEGA16U2 IC601
+L ATMEGA16U2 IC301
 U 1 1 515BCD3F
 P 6900 3250
-F 0 "IC601" H 5850 1500 60  0000 L CNN
+F 0 "IC301" H 5850 1500 60  0000 L CNN
 F 1 "ATMEGA16U2" H 5850 1400 60  0000 L CNN
 F 2 "" H 6900 3250 60  0001 C CNN

Commit message: Edit pass of footprints, cleanup symbols, etc.
Parts:
- removed X301: 12MHz KX-7 20pF, symbol CRYSTAL
- added X301: KX-7 12MHz 20pF, ~, symbol CRYSTAL_SMD
- D301: renamed from CD1206-S301; value DIODE -> CD1206-S
- F301: value PTC MF-MSMF050-2 500mA -> 500mA PTC 1812
- renumbered D301 to D302, D302 to D303
Connections:
- wire segments 101 -> 103
Changed lines of the file:
@@
-EESchema Schematic File Version 2  date Thu 11 Apr 2013 16:32:55 EST
+EESchema Schematic File Version 2  date Fri 03 May 2013 15:34:29 EST
+LIBS:freetronics_kicad_sch_lib
 LIBS:power
 LIBS:device
@@
 LIBS:contrib
 LIBS:valves
-LIBS:freetronics_kicad_sch_lib
 LIBS:EtherDue-cache
 EELAYER 24 0
@@
 Sheet 3 6
 Title ""
-Date "11 apr 2013"
+Date "3 may 2013"
 Rev ""
 Comp ""
@@
 	5550 2650 4550 2650
 Wire Wire Line
-	4150 2950 4000 2950
+	4000 2950 4800 2950
 Wire Wire Line
 	4000 2950 4000 3050
@@
 $EndComp
 $Comp
-L LED D302
+L LED D303
 U 1 1 515BD64B
 P 9300 4500
-F 0 "D302" H 9300 4600 50  0000 C CNN
+F 0 "D303" H 9300 4600 50  0000 C CNN
 F 1 "YELLOW" H 9300 4400 50  0000 C CNN
 F 2 "" H 9300 4500 60  0001 C CNN
@@
 $EndComp
 $Comp
-L LED D301
+L LED D302
 U 1 1 515BD62A
 P 9300 4200
-F 0 "D301" H 9300 4300 50  0000 C CNN
+F 0 "D302" H 9300 4300 50  0000 C CNN
 F 1 "YELLOW" H 9300 4100 50  0000 C CNN
 F 2 "" H 9300 4200 60  0001 C CNN
@@
 P 2000 3500
 F 0 "F301" H 2100 3550 40  0000 C CNN
-F 1 "PTC MF-MSMF050-2 500mA" H 2000 3350 40  0000 C CNN
+F 1 "500mA PTC 1812" H 2000 3350 40  0000 C CNN
 F 2 "" H 2000 3500 60  0001 C CNN
 F 3 "" H 2000 3500 60  0001 C CNN
@@
 F 3 "" H 4350 2750 60  0001 C CNN
 	1    4350 2750
-	0    -1   -1   0
-$EndComp
-$Comp
-L CRYSTAL X301
-U 1 1 515BCF7E
-P 4900 2950
-F 0 "X301" H 4900 3100 60  0000 C CNN
-F 1 "12MHz KX-7 20pF" H 4900 2800 60  0000 C CNN
-F 2 "" H 4900 2950 60  0001 C CNN
-F 3 "" H 4900 2950 60  0001 C CNN
-	1    4900 2950
 	0    -1   -1   0
 $EndComp
@@
 MISO
 $Comp
-L DIODE CD1206-S301
+L DIODE D301
 U 1 1 515BCE47
 P 5300 2000
-F 0 "CD1206-S301" H 5300 1850 40  0000 C CNN
-F 1 "DIODE" H 5300 1900 40  0000 C CNN
+F 0 "D301" H 5300 1850 40  0000 C CNN
+F 1 "CD1206-S" H 5300 1900 40  0000 C CNN
 F 2 "" H 5300 2000 60  0001 C CNN
 F 3 "" H 5300 2000 60  0001 C CNN
@@
 	1    0    0    -1
 $EndComp
+$Comp
+L CRYSTAL_SMD X301
+U 1 1 516F817E
+P 4900 2950
+F 0 "X301" V 5000 2850 30  0000 C CNN
+F 1 "KX-7 12MHz 20pF" H 4700 3050 30  0000 L CNN
+F 2 "~" H 4900 2950 60  0000 C CNN
+F 3 "~" H 4900 2950 60  0000 C CNN
+	1    4900 2950
+	0    1    1    0
+$EndComp
+Wire Wire Line
+	4900 2750 4900 2650
+Wire Wire Line
+	4900 3150 4900 3250
 $EndSCHEMATC

Commit message: Footprints checked, components imported to board but most not placed
Parts:
- X301: value KX-7 12MHz 20pF -> TXC 7A 12MHz 18pF
Connections:
- net labels added: XTAL1, XTAL2
Changed lines of the file:
@@
-EESchema Schematic File Version 2  date Tue 04 Jun 2013 15:53:49 EST
+EESchema Schematic File Version 2  date Thu 06 Jun 2013 09:35:07 EST
 LIBS:freetronics_kicad_sch_lib
 LIBS:power
@@
 Sheet 3 6
 Title ""
-Date "4 jun 2013"
+Date "5 jun 2013"
 Rev ""
 Comp ""
@@
 P 4900 2950
 F 0 "X301" V 5000 2850 30  0000 C CNN
-F 1 "KX-7 12MHz 20pF" H 4700 3050 30  0000 L CNN
+F 1 "TXC 7A 12MHz 18pF" H 4700 3050 30  0000 L CNN
 F 2 "~" H 4900 2950 60  0000 C CNN
 F 3 "~" H 4900 2950 60  0000 C CNN
@@
 Wire Wire Line
 	4900 3150 4900 3250
+Text Label 5550 2900 2    60   ~ 0
+XTAL1
+Text Label 5550 2650 2    60   ~ 0
+XTAL2
 $EndSCHEMATC

Commit message: Remove JP301 (breakout for 4 GPIOs from 16u2. Not routed on Due board, definitely won't fit on this board.
Parts:
- removed JP301: M02X02, symbol M02X02
Connections:
- net labels removed: 8PB4, 8PB5, 8PB6, 8PB7
- wire segments 103 -> 91
- no-connect marks 7 -> 11
Changed lines of the file:
@@
-EESchema Schematic File Version 2  date Thu 06 Jun 2013 10:22:11 EST
+EESchema Schematic File Version 2  date Thu 06 Jun 2013 10:26:06 EST
 LIBS:freetronics_kicad_sch_lib
 LIBS:power
@@
 Sheet 3 6
 Title ""
-Date "5 jun 2013"
+Date "6 jun 2013"
 Rev ""
 Comp ""
@@
 Wire Wire Line
 	4150 2750 4150 3150
-Wire Notes Line
-	8000 2000 8000 900
-Wire Notes Line
-	8000 2000 9050 2000
-Wire Notes Line
-	9050 2000 9050 900
-Wire Notes Line
-	9050 900  8000 900
-Wire Wire Line
-	8650 1200 8650 950
-Wire Wire Line
-	8650 950  8400 950
-Wire Wire Line
-	8400 950  8400 2300
-Wire Wire Line
-	8400 2300 8100 2300
-Wire Wire Line
-	8100 2500 8650 2500
-Wire Wire Line
-	8650 2500 8650 1700
 Connection ~ 5100 2400
 Wire Wire Line
@@
 Wire Wire Line
 	8100 2800 8450 2800
-Wire Wire Line
-	8100 2400 8550 2400
-Wire Wire Line
-	8550 2400 8550 1700
-Wire Wire Line
-	8100 2200 8300 2200
-Wire Wire Line
-	8300 2200 8300 1050
-Wire Wire Line
-	8300 1050 8550 1050
-Wire Wire Line
-	8550 1050 8550 1200
 Wire Wire Line
 	5150 3250 5150 2900
@@
 	0    -1   -1   0
 $EndComp
-Text Label 8400 1950 1    60   ~ 0
-8PB6
-Text Label 8550 1950 1    60   ~ 0
-8PB5
-Text Label 8650 1950 1    60   ~ 0
-8PB4
-Text Label 8300 1950 1    60   ~ 0
-8PB7
-$Comp
-L M02X02 JP301
-U 1 1 515BCEC1
-P 8650 1400
-F 0 "JP301" H 8550 1500 50  0000 C CNN
-F 1 "M02X02" H 8600 1200 40  0000 C CNN
-F 2 "" H 8650 1400 60  0001 C CNN
-F 3 "" H 8650 1400 60  0001 C CNN
-	1    8650 1400
-	0    1    -1   0
-$EndComp
 NoConn ~ 8100 2900
 Text Label 8100 2800 0    60   ~ 0
@@
 Text Label 5550 2650 2    60   ~ 0
 XTAL2
+NoConn ~ 8100 2200
+NoConn ~ 8100 2300
+NoConn ~ 8100 2400
+NoConn ~ 8100 2500
 $EndSCHEMATC
